Commit message: mimic joint

File: robotiq_85_description/urdf/robotiq_85.common.gazebo.xacro (robot description, xacro)
@@ -5,4 +5,35 @@
       <!--robotNamespace>/</robotNamespace-->
       <!--robotSimType>gazebo_ros_control/DefaultRobotHWSim</robotSimType-->
+    </plugin>
+    <!-- loading plugin: mimic joints works in gazebo now -->
+    <plugin filename="libroboticsgroup_gazebo_mimic_joint_plugin.so" name="mimic_robotiq_85_1">
+        <joint>robotiq_85_left_knuckle_joint</joint>
+        <mimicJoint>robotiq_85_right_knuckle_joint</mimicJoint>
+        <multiplier>1.0</multiplier>
+        <offset>0.0</offset>
+    </plugin>
+    <plugin filename="libroboticsgroup_gazebo_mimic_joint_plugin.so" name="mimic_robotiq_85_2">
+        <joint>robotiq_85_left_knuckle_joint</joint>
+        <mimicJoint>robotiq_85_left_inner_knuckle_joint</mimicJoint>
+        <multiplier>1.0</multiplier>
+        <offset>0.0</offset>
+    </plugin>
+    <plugin filename="libroboticsgroup_gazebo_mimic_joint_plugin.so" name="mimic_robotiq_85_3">
+        <joint>robotiq_85_left_knuckle_joint</joint>
+        <mimicJoint>robotiq_85_right_inner_knuckle_joint</mimicJoint>
+        <multiplier>1.0</multiplier>
+        <offset>0.0</offset>
+    </plugin>
+    <plugin filename="libroboticsgroup_gazebo_mimic_joint_plugin.so" name="mimic_robotiq_85_4">
+        <joint>robotiq_85_left_knuckle_joint</joint>
+        <mimicJoint>robotiq_85_left_finger_tip_joint</mimicJoint>
+        <multiplier>-1.0</multiplier>
+        <offset>0.0</offset>
+    </plugin>
+    <plugin filename="libroboticsgroup_gazebo_mimic_joint_plugin.so" name="mimic_robotiq_85_5">
+        <joint>robotiq_85_left_knuckle_joint</joint>
+        <mimicJoint>robotiq_85_right_finger_tip_joint</mimicJoint>
+        <multiplier>-1.0</multiplier>
+        <offset>0.0</offset>
     </plugin>
 <!--

File: robotiq_85_description/urdf/robotiq_85.transmission.xacro (robot description, xacro)
@@ -11,49 +11,4 @@
       </actuator>
     </transmission>
-    <transmission name="${prefix}robotiq_85_right_knuckle_trans">
-      <type>transmission_interface/SimpleTransmission</type>
-      <joint name="${prefix}robotiq_85_right_knuckle_joint">
-        <hardwareInterface>PositionJointInterface</hardwareInterface>
-      </joint>
-      <actuator name="${prefix}robotiq_85_right_knuckle_motor">
-        <mechanicalReduction>1</mechanicalReduction>
-      </actuator>
-    </transmission>
-    <transmission name="${prefix}robotiq_85_left_inner_knuckle_trans">
-      <type>transmission_interface/SimpleTransmission</type>
-      <joint name="${prefix}robotiq_85_left_inner_knuckle_joint">
-        <hardwareInterface>PositionJointInterface</hardwareInterface>
-      </joint>
-      <actuator name="${prefix}robotiq_85_left_inner_knuckle_motor">
-        <mechanicalReduction>1</mechanicalReduction>
-      </actuator>
-    </transmission>
-    <transmission name="${prefix}robotiq_85_right_inner_knuckle_trans">
-      <type>transmission_interface/SimpleTransmission</type>
-      <joint name="${prefix}robotiq_85_right_inner_knuckle_joint">
-        <hardwareInterface>PositionJointInterface</hardwareInterface>
-      </joint>
-      <actuator name="${prefix}robotiq_85_right_inner_knuckle_motor">
-        <mechanicalReduction>1</mechanicalReduction>
-      </actuator>
-    </transmission>
-    <transmission name="${prefix}robotiq_85_left_finger_tip_trans">
-      <type>transmission_interface/SimpleTransmission</type>
-      <joint name="${prefix}robotiq_85_left_finger_tip_joint">
-        <hardwareInterface>PositionJointInterface</hardwareInterface>
-      </joint>
-      <actuator name="${prefix}robotiq_85_left_finger_tip_motor">
-        <mechanicalReduction>1</mechanicalReduction>
-      </actuator>
-    </transmission>
-    <transmission name="${prefix}robotiq_85_right_finger_tip_trans">
-      <type>transmission_interface/SimpleTransmission</type>
-      <joint name="${prefix}robotiq_85_right_finger_tip_joint">
-        <hardwareInterface>PositionJointInterface</hardwareInterface>
-      </joint>
-      <actuator name="${prefix}robotiq_85_right_finger_tip_motor">
-        <mechanicalReduction>1</mechanicalReduction>
-      </actuator>
-    </transmission>
   </xacro:macro>
 </robot>

File: robotiq_85_description/urdf/robotiq_85_gripper_robot.xacro (robot description, xacro)
@@ -4,5 +4,5 @@
   <!-- common stuff -->
   <xacro:include filename="$(find robotiq_85_description)/urdf/robotiq_85.common.gazebo.xacro" />
-  <!-- ur5 -->
+  <!-- robotiq_85 -->
   <xacro:include filename="$(find robotiq_85_description)/urdf/robotiq_85_gripper.urdf.xacro" />
   <!-- arm -->
