Commit message: movit_config

File: robotiq_description/urdf/robotiq_85_gripper.urdf.xacro (robot description, xacro)
@@ -3,5 +3,5 @@
     <property name="pi" value="3.14159"/>
     <xacro:macro name="robotiq_85_gripper" params="prefix">
-        <xacro:include filename="$(find robotiq_85_description)/urdf/robotiq_85.transmission.xacro" />
+        <xacro:include filename="$(find robotiq_description)/urdf/robotiq_85.transmission.xacro" />
         <link name="${prefix}robotiq_85_root"/>
         <!--  /\  -->
@@ -16,10 +16,10 @@
             <visual>
                 <geometry>
-                    <mesh filename="package://robotiq_85_description/meshes/robotiq_85_gripper/visual/robotiq_85_base_link.dae"/>
-                </geometry>
-            </visual>
-            <collision>
-                <geometry>
-                    <mesh filename="package://robotiq_85_description/meshes/robotiq_85_gripper/collision/robotiq_85_base_link.stl"/>
+                    <mesh filename="package://robotiq_description/meshes/robotiq_85/visual/robotiq_85_base_link.dae"/>
+                </geometry>
+            </visual>
+            <collision>
+                <geometry>
+                    <mesh filename="package://robotiq_description/meshes/robotiq_85/collision/robotiq_85_base_link.stl"/>
                 </geometry>
             </collision>
@@ -54,10 +54,10 @@
             <visual>
                 <geometry>
-                    <mesh filename="package://robotiq_85_description/meshes/robotiq_85_gripper/visual/robotiq_85_knuckle_link.dae"/>
-                </geometry>
-            </visual>
-            <collision>
-                <geometry>
-                    <mesh filename="package://robotiq_85_description/meshes/robotiq_85_gripper/collision/robotiq_85_knuckle_link.stl"/>
+                    <mesh filename="package://robotiq_description/meshes/robotiq_85/visual/robotiq_85_knuckle_link.dae"/>
+                </geometry>
+            </visual>
+            <collision>
+                <geometry>
+                    <mesh filename="package://robotiq_description/meshes/robotiq_85/collision/robotiq_85_knuckle_link.stl"/>
                 </geometry>
             </collision>
@@ -73,10 +73,10 @@
             <visual>
                 <geometry>
-                    <mesh filename="package://robotiq_85_description/meshes/robotiq_85_gripper/visual/robotiq_85_knuckle_link.dae"/>
-                </geometry>
-            </visual>
-            <collision>
-                <geometry>
-                    <mesh filename="package://robotiq_85_description/meshes/robotiq_85_gripper/collision/robotiq_85_knuckle_link.stl"/>
+                    <mesh filename="package://robotiq_description/meshes/robotiq_85/visual/robotiq_85_knuckle_link.dae"/>
+                </geometry>
+            </visual>
+            <collision>
+                <geometry>
+                    <mesh filename="package://robotiq_description/meshes/robotiq_85/collision/robotiq_85_knuckle_link.stl"/>
                 </geometry>
             </collision>
@@ -110,10 +110,10 @@
             <visual>
                 <geometry>
-                    <mesh filename="package://robotiq_85_description/meshes/robotiq_85_gripper/visual/robotiq_85_finger_link.dae"/>
-                </geometry>
-            </visual>
-            <collision>
-                <geometry>
-                    <mesh filename="package://robotiq_85_description/meshes/robotiq_85_gripper/collision/robotiq_85_finger_link.stl"/>
+                    <mesh filename="package://robotiq_description/meshes/robotiq_85/visual/robotiq_85_finger_link.dae"/>
+                </geometry>
+            </visual>
+            <collision>
+                <geometry>
+                    <mesh filename="package://robotiq_description/meshes/robotiq_85/collision/robotiq_85_finger_link.stl"/>
                 </geometry>
             </collision>
@@ -129,10 +129,10 @@
             <visual>
                 <geometry>
-                    <mesh filename="package://robotiq_85_description/meshes/robotiq_85_gripper/visual/robotiq_85_finger_link.dae"/>
-                </geometry>
-            </visual>
-            <collision>
-                <geometry>
-                    <mesh filename="package://robotiq_85_description/meshes/robotiq_85_gripper/collision/robotiq_85_finger_link.stl"/>
+                    <mesh filename="package://robotiq_description/meshes/robotiq_85/visual/robotiq_85_finger_link.dae"/>
+                </geometry>
+            </visual>
+            <collision>
+                <geometry>
+                    <mesh filename="package://robotiq_description/meshes/robotiq_85/collision/robotiq_85_finger_link.stl"/>
                 </geometry>
             </collision>
@@ -168,10 +168,10 @@
             <visual>
                 <geometry>
-                    <mesh filename="package://robotiq_85_description/meshes/robotiq_85_gripper/visual/robotiq_85_inner_knuckle_link.dae"/>
-                </geometry>
-            </visual>
-            <collision>
-                <geometry>
-                    <mesh filename="package://robotiq_85_description/meshes/robotiq_85_gripper/collision/robotiq_85_inner_knuckle_link.stl"/>
+                    <mesh filename="package://robotiq_description/meshes/robotiq_85/visual/robotiq_85_inner_knuckle_link.dae"/>
+                </geometry>
+            </visual>
+            <collision>
+                <geometry>
+                    <mesh filename="package://robotiq_description/meshes/robotiq_85/collision/robotiq_85_inner_knuckle_link.stl"/>
                 </geometry>
             </collision>
@@ -187,10 +187,10 @@
             <visual>
                 <geometry>
-                    <mesh filename="package://robotiq_85_description/meshes/robotiq_85_gripper/visual/robotiq_85_inner_knuckle_link.dae"/>
-                </geometry>
-            </visual>
-            <collision>
-                <geometry>
-                    <mesh filename="package://robotiq_85_description/meshes/robotiq_85_gripper/collision/robotiq_85_inner_knuckle_link.stl"/>
+                    <mesh filename="package://robotiq_description/meshes/robotiq_85/visual/robotiq_85_inner_knuckle_link.dae"/>
+                </geometry>
+            </visual>
+            <collision>
+                <geometry>
+                    <mesh filename="package://robotiq_description/meshes/robotiq_85/collision/robotiq_85_inner_knuckle_link.stl"/>
                 </geometry>
             </collision>
@@ -226,10 +226,10 @@
             <visual>
                 <geometry>
-                    <mesh filename="package://robotiq_85_description/meshes/robotiq_85_gripper/visual/robotiq_85_finger_tip_link.dae"/>
-                </geometry>
-            </visual>
-            <collision>
-                <geometry>
-                    <mesh filename="package://robotiq_85_description/meshes/robotiq_85_gripper/collision/robotiq_85_finger_tip_link.stl"/>
+                    <mesh filename="package://robotiq_description/meshes/robotiq_85/visual/robotiq_85_finger_tip_link.dae"/>
+                </geometry>
+            </visual>
+            <collision>
+                <geometry>
+                    <mesh filename="package://robotiq_description/meshes/robotiq_85/collision/robotiq_85_finger_tip_link.stl"/>
                 </geometry>
             </collision>
@@ -245,10 +245,10 @@
             <visual>
                 <geometry>
-                    <mesh filename="package://robotiq_85_description/meshes/robotiq_85_gripper/visual/robotiq_85_finger_tip_link.dae"/>
-                </geometry>
-            </visual>
-            <collision>
-                <geometry>
-                    <mesh filename="package://robotiq_85_description/meshes/robotiq_85_gripper/collision/robotiq_85_finger_tip_link.stl"/>
+                    <mesh filename="package://robotiq_description/meshes/robotiq_85/visual/robotiq_85_finger_tip_link.dae"/>
+                </geometry>
+            </visual>
+            <collision>
+                <geometry>
+                    <mesh filename="package://robotiq_description/meshes/robotiq_85/collision/robotiq_85_finger_tip_link.stl"/>
                 </geometry>
             </collision>

File: robotiq_description/urdf/robotiq_85_gripper.xacro (robot description, xacro)
@@ -1,5 +1,5 @@
 <?xml version="1.0" ?>
 <robot name="robotiq_85_gripper" xmlns:xacro="http://ros.org/wiki/xacro">
-    <xacro:include filename="$(find robotiq_85_description)/urdf/robotiq_85_gripper.urdf.xacro" />
+    <xacro:include filename="$(find robotiq_description)/urdf/robotiq_85_gripper.urdf.xacro" />
     <xacro:robotiq_85_gripper prefix=""/>
 </robot>

File: robotiq_description/urdf/robotiq_85_gripper_robot.xacro (robot description, xacro)
@@ -3,7 +3,7 @@
        name="robotiq_85_gripper" >
   <!-- common stuff -->
-  <xacro:include filename="$(find robotiq_85_description)/urdf/robotiq_85.common.gazebo.xacro" />
+  <xacro:include filename="$(find robotiq_description)/urdf/robotiq_85.common.gazebo.xacro" />
   <!-- robotiq_85 -->
-  <xacro:include filename="$(find robotiq_85_description)/urdf/robotiq_85_gripper.urdf.xacro" />
+  <xacro:include filename="$(find robotiq_description)/urdf/robotiq_85_gripper.urdf.xacro" />
   <!-- arm -->
   <xacro:robotiq_85_gripper prefix=""/>
